File: FABI3 - IMU Addon/FABI3 - IMU Addon.kicad_sch (KiCad schematic)
At the start: 10 parts, among them J1 RJ25, U1 ICM-42670-P, U2 MIC94310

Commit message: Add files via upload
Other:
- note added: "300mA"
Changed lines of the file:
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@@
+    (effects (font (size 1.27 1.27)) (justify left bottom))
+  )
+  (text "300mA" (at 30.48 93.98 0)
     (effects (font (size 1.27 1.27)) (justify left bottom))
   )
